File: board/rfid-player/rfid-player.sch (KiCad schematic (older format))
At the start: 22 parts

Commit message: Board fixes
Parts:
- R10, R3, R4, R6, R7, R9: value R -> 2k2
- R11, R5, R8: value R -> 1k
Connections:
- net D10: now also R3.1; no longer R3.2, R4.1
- net D11: now also R9.1; no longer R6.2, R7.1
- net D13: now also R6.1; no longer R10.1, R9.2
- net GND: now also RVol1.3; no longer RVol1.1
- net MOSI: now also R6.2, R7.1; no longer R9.1
- net SCK: now also R10.1, R9.2; no longer R6.1
- net SDA: now also R3.2, R4.1; no longer R3.1
- net at AMP1.1 (Pin_1), R12.1, R13.2: now also RVol1.1; no longer RVol1.3
Changed lines of the file:
@@
 U 1 1 5FC916AC
 P 4250 4900
-F 0 "R4" V 4400 4950 50  0000 C CNN
-F 1 "R" V 4400 4850 50  0000 C CNN
+F 0 "R4" V 4350 4950 50  0000 C CNN
+F 1 "2k2" V 4350 4800 50  0000 C CNN
 F 2 "Resistors_THT:R_Axial_DIN0204_L3.6mm_D1.6mm_P5.08mm_Horizontal" V 4180 4900 50  0001 C CNN
 F 3 "~" H 4250 4900 50  0001 C CNN
@@
 U 1 1 5FC91BBF
 P 4250 5200
-F 0 "R5" V 4400 5250 50  0000 C CNN
-F 1 "R" V 4400 5150 50  0000 C CNN
+F 0 "R5" V 4350 5200 50  0000 C CNN
+F 1 "1k" V 4350 5050 50  0000 C CNN
 F 2 "Resistors_THT:R_Axial_DIN0204_L3.6mm_D1.6mm_P5.08mm_Horizontal" V 4180 5200 50  0001 C CNN
 F 3 "~" H 4250 5200 50  0001 C CNN
@@
 U 1 1 5FC91E0F
 P 4250 4600
-F 0 "R3" V 4400 4650 50  0000 C CNN
-F 1 "R" V 4400 4550 50  0000 C CNN
+F 0 "R3" V 4350 4750 50  0000 C CNN
+F 1 "2k2" V 4350 4600 50  0000 C CNN
 F 2 "Resistors_THT:R_Axial_DIN0204_L3.6mm_D1.6mm_P5.08mm_Horizontal" V 4180 4600 50  0001 C CNN
 F 3 "~" H 4250 4600 50  0001 C CNN
@@
 U 1 1 5FC952BA
 P 4550 4900
-F 0 "R7" V 4700 4950 50  0000 C CNN
-F 1 "R" V 4700 4850 50  0000 C CNN
+F 0 "R7" V 4650 4950 50  0000 C CNN
+F 1 "2k2" V 4650 4800 50  0000 C CNN
 F 2 "Resistors_THT:R_Axial_DIN0204_L3.6mm_D1.6mm_P5.08mm_Horizontal" V 4480 4900 50  0001 C CNN
 F 3 "~" H 4550 4900 50  0001 C CNN
@@
 U 1 1 5FC952C0
 P 4550 5200
-F 0 "R8" V 4700 5250 50  0000 C CNN
-F 1 "R" V 4700 5150 50  0000 C CNN
+F 0 "R8" V 4650 5200 50  0000 C CNN
+F 1 "1k" V 4650 5050 50  0000 C CNN
 F 2 "Resistors_THT:R_Axial_DIN0204_L3.6mm_D1.6mm_P5.08mm_Horizontal" V 4480 5200 50  0001 C CNN
 F 3 "~" H 4550 5200 50  0001 C CNN
@@
 U 1 1 5FC952C6
 P 4550 4600
-F 0 "R6" V 4700 4650 50  0000 C CNN
-F 1 "R" V 4700 4550 50  0000 C CNN
+F 0 "R6" V 4650 4750 50  0000 C CNN
+F 1 "2k2" V 4650 4600 50  0000 C CNN
 F 2 "Resistors_THT:R_Axial_DIN0204_L3.6mm_D1.6mm_P5.08mm_Horizontal" V 4480 4600 50  0001 C CNN
 F 3 "~" H 4550 4600 50  0001 C CNN
@@
 U 1 1 5FC95F5C
 P 4850 4900
-F 0 "R10" V 5000 4950 50  0000 C CNN
-F 1 "R" V 5000 4850 50  0000 C CNN
+F 0 "R10" V 4950 4950 50  0000 C CNN
+F 1 "2k2" V 4950 4800 50  0000 C CNN
 F 2 "Resistors_THT:R_Axial_DIN0204_L3.6mm_D1.6mm_P5.08mm_Horizontal" V 4780 4900 50  0001 C CNN
 F 3 "~" H 4850 4900 50  0001 C CNN
@@
 U 1 1 5FC95F62
 P 4850 5200
-F 0 "R11" V 5000 5250 50  0000 C CNN
-F 1 "R" V 5000 5150 50  0000 C CNN
+F 0 "R11" V 4950 5200 50  0000 C CNN
+F 1 "1k" V 4950 5050 50  0000 C CNN
 F 2 "Resistors_THT:R_Axial_DIN0204_L3.6mm_D1.6mm_P5.08mm_Horizontal" V 4780 5200 50  0001 C CNN
 F 3 "~" H 4850 5200 50  0001 C CNN
@@
 U 1 1 5FC95F68
 P 4850 4600
-F 0 "R9" V 5000 4650 50  0000 C CNN
-F 1 "R" V 5000 4550 50  0000 C CNN
+F 0 "R9" V 4950 4750 50  0000 C CNN
+F 1 "2k2" V 4950 4600 50  0000 C CNN
 F 2 "Resistors_THT:R_Axial_DIN0204_L3.6mm_D1.6mm_P5.08mm_Horizontal" V 4780 4600 50  0001 C CNN
 F 3 "~" H 4850 4600 50  0001 C CNN
@@
 NoConn ~ 5500 5300
 Text GLabel 4250 4450 1    50   Input ~ 0
-SDA
-Text GLabel 4550 4450 1    50   Input ~ 0
-SCK
+D10
 Text GLabel 4850 4450 1    50   Input ~ 0
-MOSI
+D11
 Text GLabel 6300 3550 0    50   Input ~ 0
-D10
-Text GLabel 4250 4750 0    50   Input ~ 0
 D10
 Text GLabel 6300 3650 0    50   Input ~ 0
 D11
 Text GLabel 4550 4750 0    50   Input ~ 0
-D11
+MOSI
 Text GLabel 6300 3850 0    50   Input ~ 0
 D13
 Text GLabel 4850 4750 0    50   Input ~ 0
-D13
+SCK
 $Comp
 L Device:R R12
@@
 F 3 "~" H 7050 5150 50  0001 C CNN
 	1    7050 5150
-	0    1    -1   0
+	0    -1   -1   0
 $EndComp
 Wire Wire Line
@@
 $EndComp
 NoConn ~ 7750 3400
+Text GLabel 4550 4450 1    50   Input ~ 0
+D13
+Text GLabel 4250 4750 0    50   Input ~ 0
+SDA
 $EndSCHEMATC
